File: VIPR_PCB/PiHAT_SSR_V4/PiHAT_SSR_V4.brd (EAGLE design)
At the start: 65 x 68.7 mm, 47 parts, among them CN1 M12_8PIN_CODE_A, J10 GPIO_5 (OUT), J11 GPIO_17 (IN), J12 GPIO_12, J8 GPIO_13 (OUT), J9 GPIO_6 (OUT)

Commit message: Add files via upload
Parts:
- R10, R8, R9: value (none) -> 12; device rcl:R2512 -> rcl:R1210
- moved C5 21.0 mm to (11.9, 3.60), turned to 180 degrees
- moved C3 20.1 mm to (11.9, 6.10), turned to 180 degrees
- moved R10 10.5 mm to (38.4, 40.8), turned to 0 degrees
- moved R9 9.65 mm to (50.4, 39.8), turned to 0 degrees
- moved AUML1 8.64 mm to (23.3, 23.3), turned to 0 degrees
- moved R8 7.29 mm to (60.1, 38.0), turned to 0 degrees
- moved D4 6.39 mm to (38.1, 43.9), turned to 0 degrees
- moved D3 5.17 mm to (50.4, 42.9), turned to 0 degrees
- moved J6 4.18 mm to (43.4, 33.3)
- moved D1 3.67 mm to (41.0, 28.3)
- moved D2 1.90 mm to (60.1, 40.9), turned to 0 degrees
- moved C6 1.39 mm to (35.2, 21.8), turned to 180 degrees
- moved J9 0.54 mm to (42.5, 59.8)
- moved C1 0.51 mm to (34.6, 15.5)
- moved J4 0.36 mm to (53.8, 60.8)
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Connections:
- net 12V_PWR_IN: now also CN1.P$2; no longer CN1.P$6
- net GND: now also CN1.P$3; no longer CN1.P$7
- net SOL_1: now also CN1.P$1, D4.P$1, SSR3.P$5, SSR3.P$8; no longer CN1.P$5, R10.1, SSR3.P$6, SSR3.P$7
- net SOL_12V: now also CN1.P$5, R10.1, R8.1, R9.1; no longer CN1.P$2, SSR1.P$5, SSR1.P$8, SSR2.P$5, SSR2.P$8, SSR3.P$5, SSR3.P$8
- net SOL_2: now also CN1.P$6, D2.P$1, SSR1.P$5, SSR1.P$8; no longer CN1.P$3, R8.1, SSR1.P$6, SSR1.P$7
- net SOL_3: now also CN1.P$7, D3.P$1, SSR2.P$5, SSR2.P$8; no longer CN1.P$4, R9.1, SSR2.P$6, SSR2.P$7
- net SOL_GND: now also CN1.P$4, SSR1.P$6, SSR1.P$7, SSR2.P$6, SSR2.P$7, SSR3.P$6, SSR3.P$7; no longer CN1.P$1, D2.P$1, D3.P$1, D4.P$1
Routing:
- net SOL_GND: track 8.30 -> 16.3 mm
- net SOL_2: track 51.4 -> 57.0 mm
- net SOL_3: track 49.7 -> 54.4 mm
- net 12V_PWR_IN: track 17.8 -> 20.7 mm
- net GND: track 45.0 -> 43.3 mm
- net N$1: track 4.53 -> 2.96 mm
- net N$7: track 4.53 -> 3.16 mm
- net N$3: track 4.53 -> 3.16 mm
- net GPIO_17: track 25.5 -> 26.9 mm
- net ENABLE_SOL_12V: track 55.9 -> 54.9 mm, vias 2 -> 0
- net PWR_IN_12V_D: track 30.7 -> 31.5 mm
- net GPIO_13: track 18.0 -> 18.6 mm
Other:
- board text added: "PiHAT_SSRelay_V4_3_31_2020"
- board text removed: "PiHAT_SSRelay_V4_3_23_2020"
