File: VIPR_PCB/PiHAT_SSR_V4/PiHAT_SSR_V4.sch (EAGLE design)
At the start: 47 parts, among them CN1 M12_8PIN_CODE_A, J10 GPIO_5 (OUT), J11 GPIO_17 (IN), J12 GPIO_12, J8 GPIO_13 (OUT), J9 GPIO_6 (OUT)

Commit message: Add files via upload
Parts:
- R10, R8, R9: value (none) -> 12; device rcl:R-US_R2512 -> rcl:R-US_R1210
Connections:
- net 12V_PWR_IN: now also CN1.P$2; no longer CN1.P$6
- net GND: now also CN1.P$3; no longer CN1.P$7
- net SOL_1: now also CN1.P$1, D4.A, SSR3.VLOAD(5), SSR3.VLOAD(8); no longer CN1.P$5, R10.1, SSR3.GND(6), SSR3.GND(7)
- net SOL_12V: now also CN1.P$5, R10.1, R8.1, R9.1; no longer CN1.P$2, SSR1.VLOAD(5), SSR1.VLOAD(8), SSR2.VLOAD(5), SSR2.VLOAD(8), SSR3.VLOAD(5), SSR3.VLOAD(8)
- net SOL_2: now also CN1.P$6, D2.A, SSR1.VLOAD(5), SSR1.VLOAD(8); no longer CN1.P$3, R8.1, SSR1.GND(6), SSR1.GND(7)
- net SOL_3: now also CN1.P$7, D3.A, SSR2.VLOAD(5), SSR2.VLOAD(8); no longer CN1.P$4, R9.1, SSR2.GND(6), SSR2.GND(7)
- net SOL_GND: now also CN1.P$4, SSR1.GND(6), SSR1.GND(7), SSR2.GND(6), SSR2.GND(7), SSR3.GND(6), SSR3.GND(7); no longer CN1.P$1, D2.A, D3.A, D4.A
Other:
- note added: "DC Parallel Load Connection (C): rated for 6 A continuous"
- note added: "List of GPIOs used: ------------------------------------------------- GPIO 12 - Not used, pad available (no relay) GPIO 13 - Middle/Main solenoid/air-knife GPIO 6 - Neighboring right-side solenoid/air-knife GPIO 5 - Neighboring left-side solenoid/air knifel"
- note added: "Pinouts for 8-pin M12 Connector: ---------------------------------------------------------------------------------------------------------- 1. Solenoid 1 GPIO 5 (12VDC SS-Relay output: left side neighbor switched air-knife) 2. Raspberry Pi 12V power, to be stepped down to 5V with regulators 3. Raspberry Pi GND 4. Solenoid isolated GND 5. Solenoid 12V 6. Solenoid 2 GPIO 13 (12VDC SS-Relay output: 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"
- note added: "Reverse biased schottky diode in parallel with the solenoid to act as a flyback diode for circuit protection from voltage spikes caused by inductive loads."
- note added: "SSRelay 1 (SOL_2) - Middle/main switched solenoid/air-knife"
- note added: "SSRelay 2 (SOL_3) - Neighboring right-side switched solenoid/air-knife"
- note added: "SSRelay 3 (SOL_1) - Neighboring left-side switched solenoid/air-knife"
- note added: "Solenoids connected in a low-side switch configuration. Meaning solenoids are always connected to 12V and relays will handle connection to GND"
- note removed: "DC Parallel Load Connection: rated for 1000 mA continuous"
- note removed: "List of GPIOs used: ------------------------------------------------- GPIO 26 - Indicator LED GPIO 12 - Neighboring left-side solenoid/air-knife GPIO 13 - Middle/Main solenoid/air-knife GPIO 6 - Neighboring right-side solenoid/air-knife GPIO 5 - Clean/cooling air solenoid control"
- note removed: "Pinouts for 8-pin M12 Connector: ---------------------------------------------------------------------------------------------------------- 1. Solenoid isolated GND 2. Solenoid 12V 3. Solenoid 2 (12VDC SS-Relay output: main/middle switched air-knife) 4. Solenoid 1 (12VDC SS-Relay output: left side neighbor switched air-knife) 5. Solenoid 3 (12VDC SS-Relay output: right side neighbor switched air-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"
- note removed: "SSRelay 1 - Middle/main switched solenoid/air-knife"
- note removed: "SSRelay 2 - Neighboring right-side switched solenoid/air-knife"
- note removed: "SSRelay 3 - Neighboring left-side switched solenoid/air-knife"
- note removed: "Solenoids connected in a high-side switch configuration. Meaning solenoids are always connected to ground and relays will handle connection to 12V"
- moved on the sheet: D2, D3, D4, R10, R8, R9
